File: electrical/mechanical_switch/RB_Switch.kicad_pcb (KiCad board)
At the start: 4 copper layers, 115 x 38 mm, 33 parts, among them SW1 SW_TH_Tactile_Omron_B3F-10xx, SW2 SW_TH_Tactile_Omron_B3F-10xx, SW3 SW_TH_Tactile_Omron_B3F-10xx, U1 ESP32-S2-MINI-1

Commit message: corrected gerber files
Parts:
- moved C1 112.4 mm to (122.0, 86.0)
- moved C10 112.4 mm to (164.0, 113.0)
- moved C11 112.4 mm to (170.0, 113.0)
- moved C2 112.4 mm to (128.0, 86.0)
- moved C3 112.4 mm to (140.0, 86.0)
- moved C4 112.4 mm to (152.0, 86.0)
- moved C5 112.4 mm to (140.0, 113.0)
- moved C6 112.4 mm to (146.0, 113.0)
- moved C7 112.4 mm to (152.0, 113.0)
- moved C8 112.4 mm to (110.0, 113.0)
- moved C9 112.4 mm to (158.0, 113.0)
- moved D1 112.4 mm to (158.0, 86.0)
- moved J_BAT 112.4 mm to (116.0, 86.0)
- moved J_USB 112.4 mm to (84.0, 99.0), turned to -90 degrees
- moved L1 112.4 mm to (134.0, 86.0)
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
Commit message: editing pcb
Parts:
- moved L1 35.4 mm to (98.6, 86.0), turned to 90 degrees
- turned J_BAT to 180 degrees
- turned U1 to -90 degrees
Routing:
- net L_B: track 32.9 -> 5.10 mm
- net L_A: track 29.9 -> 5.10 mm, vias 0 -> 2
- net SW2_NET: track 71.5 -> 96.3 mm, vias 4 -> 2
- net SW3_NET: track 50.4 -> 71.0 mm, vias 0 -> 2
- net USB_DP: track 104.9 -> 85.4 mm, vias 0 -> 3
- net USB_DM: track 105.4 -> 86.1 mm, vias 4 -> 3
- net BOOT_NET: track 49.5 -> 68.4 mm, vias 4 -> 3
- net USB_CC1: track 31.7 -> 45.8 mm
- net SW1_NET: track 94.7 -> 105.3 mm, vias 0 -> 2
- net EN_NET: track 87.8 -> 98.1 mm, vias 0 -> 3
- net VBAT_SENSE: track 96.4 -> 104.7 mm, vias 6 -> 4
- net USB_CC2: track 40.3 -> 47.3 mm, vias 0 -> 2
- net VBUS: track 74.2 -> 81.0 mm, vias 0 -> 4
- net VBAT: track 67.8 -> 73.6 mm, vias 12 -> 6
- net CHG_STAT: track 48.4 -> 50.6 mm
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