File: electrical/mechanical_switch/RB_Switch.kicad_pcb (KiCad board)
At the start: 4 copper layers, 115 x 38 mm, 33 parts, among them SW1 SW_TH_Tactile_Omron_B3F-10xx, SW2 SW_TH_Tactile_Omron_B3F-10xx, SW3 SW_TH_Tactile_Omron_B3F-10xx, U1 ESP32-S2-MINI-1

Commit message: Optimize switch routing and improve regulator fanout
Routing:
- net SW1_NET: track 110.3 -> 45.0 mm
- net SW2_NET: track 100.5 -> 52.5 mm
- net SW3_NET: track 71.0 -> 52.5 mm
Changed lines of the file:
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@@
-	)
-	(segment
-		(start 125.5 100.25)
-		(end 156.25 100.25)
-		(width 0.2)
-		(layer "In2.Cu")
-		(net "SW1_NET")
 	)
 	(segment
@@
 	)
 	(segment
-		(start 156.25 100.25)
-		(end 156.25 104)
-		(width 0.2)
-		(layer "In2.Cu")
-		(net "SW1_NET")
-	)
-	(segment
-		(start 101 99)
-		(end 124.75 99)
-		(width 0.2)
-		(layer "In2.Cu")
-		(net "SW1_NET")
-	)
-	(segment
 		(start 156.5 104.5)
 		(end 157 104.5)
@@
 	)
 	(segment
-		(start 126 99)
-		(end 149.75 99)
-		(width 0.2)
-		(layer "In2.Cu")
-		(net "SW2_NET")
-	)
-	(segment
 		(start 170.75 97.75)
 		(end 170.75 91.5)
@@
 		(net "SW2_NET")
 	)
-	(segment
-		(start 150.5 97.75)
-		(end 170.75 97.75)
-		(width 0.2)
-		(layer "In2.Cu")
-		(net "SW2_NET")
-	)
 	(via
 		(at 169.45 93.05)
@@
 			(back no)
 		)
-		(net "SW3_NET")
-	)
-	(segment
-		(start 168.75 98.75)
-		(end 169 98.75)
-		(width 0.2)
-		(layer "B.Cu")
 		(net "SW3_NET")
 	)
@@
 	)
 	(segment
-		(start 151 99)
-		(end 168.75 99)
-		(width 0.2)
-		(layer "B.Cu")
-		(net "SW3_NET")
-	)
-	(segment
 		(start 170 105.5)
 		(end 170 98.5)
@@
 	)
 	(segment
-		(start 169 98.75)
-		(end 169 98.5)
-		(width 0.2)
-		(layer "B.Cu")
-		(net "SW3_NET")
-	)
-	(segment
 		(start 170.25 113)
 		(end 170.25 113.5)
-		(width 0.2)
-		(layer "B.Cu")
-		(net "SW3_NET")
-	)
-	(segment
-		(start 168.75 99)
-		(end 168.75 98.75)
 		(width 0.2)
 		(layer "B.Cu")
@@
 	)
 	(segment
-		(start 124.75 99)
-		(end 124.75 101)
-		(width 0.2)
-		(layer "In2.Cu")
-		(net "SW1_NET")
-	)
-	(segment
-		(start 124.75 101)
-		(end 125.5 101)
-		(width 0.2)
-		(layer "In2.Cu")
-		(net "SW1_NET")
-	)
-	(segment
-		(start 125.5 101)
-		(end 125.5 100.25)
-		(width 0.2)
-		(layer "In2.Cu")
-		(net "SW1_NET")
-	)
-	(segment
-		(start 149.75 99)
-		(end 149.75 97.75)
-		(width 0.2)
-		(layer "In2.Cu")
-		(net "SW2_NET")
-	)
-	(segment
-		(start 149.75 97.75)
-		(end 150.5 97.75)
-		(width 0.2)
-		(layer "In2.Cu")
-		(net "SW2_NET")
-	)
-	(segment
 		(start 150.5 97.75)
 		(end 150.5 98)
@@
 	)
 	(segment
-		(start 124.75 99)
-		(end 124.75 101)
-		(width 0.2)
-		(layer "In2.Cu")
-		(net "SW1_NET")
-	)
-	(segment
-		(start 124.75 101)
-		(end 125.5 101)
-		(width 0.2)
-		(layer "In2.Cu")
-		(net "SW1_NET")
-	)
-	(segment
-		(start 125.5 101)
-		(end 125.5 100.25)
-		(width 0.2)
-		(layer "In2.Cu")
-		(net "SW1_NET")
-	)
-	(segment
-		(start 149.75 99)
-		(end 149.75 97.75)
-		(width 0.2)
-		(layer "In2.Cu")
-		(net "SW2_NET")
-	)
-	(segment
-		(start 149.75 97.75)
-		(end 150.5 97.75)
-		(width 0.2)
-		(layer "In2.Cu")
-		(net "SW2_NET")
-	)
-	(segment
 		(start 150.5 97.75)
 		(end 150.5 98)
@@
 	)
 )
+	(segment
+		(start 101 99)
+		(end 101 101.5)
+		(width 0.2)
+		(layer "In2.Cu")
+		(net "SW1_NET")
+	)
+	(segment
+		(start 101 101.5)
+		(end 156.25 101.5)
+		(width 0.2)
+		(layer "In2.Cu")
+		(net "SW1_NET")
+	)
+	(segment
+		(start 156.25 101.5)
+		(end 156.25 104)
+		(width 0.2)
+		(layer "In2.Cu")
+		(net "SW1_NET")
+	)
+	(segment
+		(start 126 99)
+		(end 126 96.5)
+		(width 0.2)
+		(layer "In2.Cu")
+		(net "SW2_NET")
+	)
+	(segment
+		(start 126 96.5)
+		(end 170.75 96.5)
+		(width 0.2)
+		(layer "In2.Cu")
+		(net "SW2_NET")
+	)
+	(segment
+		(start 170.75 96.5)
+		(end 170.75 97.75)
+		(width 0.2)
+		(layer "In2.Cu")
+		(net "SW2_NET")
+	)
+	(segment
+		(start 151 99)
+		(end 151 101.5)
+		(width 0.2)
+		(layer "B.Cu")
+		(net "SW3_NET")
+	)
+	(segment
+		(start 151 101.5)
+		(end 168.5 101.5)
+		(width 0.2)
+		(layer "B.Cu")
+		(net "SW3_NET")
+	)
+	(segment
+		(start 168.5 101.5)
+		(end 168.5 98.5)
+		(width 0.2)
+		(layer "B.Cu")
+		(net "SW3_NET")
+	)
+	(segment
+		(start 168.5 98.5)
+		(end 169 98.5)
+		(width 0.2)
+		(layer "B.Cu")
+		(net "SW3_NET")
+	)
+	(segment
+		(start 102.6 87)
+		(end 102.5 87)
+		(width 0.2)
+		(layer "F.Cu")
+		(net "VBAT")
+	)
+	(segment
+		(start 105.4 86)
+		(end 106 86)
+		(width 0.2)
+		(layer "F.Cu")
+		(net "VBAT")
+	)
+	(segment
+		(start 102.6 85.5)
+		(end 100.8 85.5)
+		(width 0.2)
+		(layer "F.Cu")
+		(net "L_B")
+	)
+	(segment
+		(start 102.6 86.5)
+		(end 100.8 86.5)
+		(width 0.2)
+		(layer "F.Cu")
+		(net "L_A")
+	)
+	(segment
+		(start 102.6 85)
+		(end 102.6 83.5)
+		(width 0.2)
+		(layer "F.Cu")
+		(net "V3V3")
+	)
+	(segment
+		(start 102.6 83.5)
+		(end 101 83.5)
+		(width 0.2)
+		(layer "F.Cu")
+		(net "V3V3")
+	)
