File: electrical/mechanical_switch/RB_Switch.kicad_sch (KiCad schematic)
At the start: 31 parts, among them SW1 B3F-10xx, SW2 B3F-10xx, SW3 B3F-10xx, U1 ESP32-S3-MINI-1

Commit message: corrected gerber files
Other:
- company: (none) -> Michael Ryan Hunsaker, M.Ed., Ph.D.
- title: (none) -> RB SWITCH Schematic

Commit message: Reconcile U1 schematic value with production module
Parts:
- U1: value ESP32-S3-MINI-1 -> ESP32-S3-MINI-1-N4R2
Changed lines of the file:
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@@
 			)
 		)
-		(property "Value" "ESP32-S3-MINI-1"
+		(property "Value" "ESP32-S3-MINI-1-N4R2"
 			(at 124.47 113.09 0)
 			(show_name no)
