File: electrical/mechanical_switch/RB_Switch.kicad_sch (KiCad schematic)
At the start: 31 parts, among them SW1 B3F-10xx, SW2 B3F-10xx, SW3 B3F-10xx, U1 ESP32-S3-MINI-1-N4R2

Commit message: clean gerners now
Parts:
- SW1, SW2, SW3: value B3F-10xx -> B3F-100x; footprint Button_Switch_THT:SW_TH_Tactile_Omron_B3F-10xx -> Button_Switch_THT:SW_TH_Tactile_Omron_B3F-100x
- renumbered J_BAT to J_BAT1, J_USB to J_USB1, SW_BOOT to SW_BOOT1, SW_RST to SW_RST1, U_CHG to U_CHG1
Connections:
- net GND: now also J_USB1.SH (SHIELD); no longer J_USB1.S1 (SHIELD)
