File: electrical/mechanical_switch/old/RB_Switch.kicad_pcb (KiCad board)
At the start: 4 copper layers, 115 x 38 mm, 33 parts, among them SW1 SW_TH_Tactile_Omron_B3F-10xx, SW2 SW_TH_Tactile_Omron_B3F-10xx, SW3 SW_TH_Tactile_Omron_B3F-10xx, U1 ESP32-S2-MINI-1

Commit message: fixed schematic and pcb errors
Parts:
- C1, C10, C11, C2, C3, C4, C5, C6, C7, C8, C9: footprint Capacitor_SMD:C_0603_1608Metric -> C_0603_1608Metric
- D1: footprint LED_SMD:LED_0603_1608Metric -> LED_0603_1608Metric
- J_BAT: footprint Connector_JST:JST_PH_S2B-PH-K_1x02_P2.00mm_Horizontal -> JST_PH_S2B-PH-K_1x02_P2.00mm_Horizontal
- J_USB: footprint Connector_USB:USB_C_Receptacle_GCT_USB4105-xx-A_16P_TopMnt_Horizontal -> USB_C_Receptacle_GCT_USB4105-xx-A_16P_TopMnt_Horizontal
- L1: footprint Inductor_SMD:L_Bourns-SRN4018 -> L_Bourns-SRN4018
- MH1, MH2: footprint MountingHole:MountingHole_4.3mm_M4 -> MountingHole_4.3mm_M4
- R1, R2, R3, R4, R5, R6, R7, R8: footprint Resistor_SMD:R_0603_1608Metric -> R_0603_1608Metric
- REG1: value TPS63001DRCR -> Texas_DRC0010J_ThermalVias; footprint Package_SON:Texas_DRC0010J -> Texas_DRC0010J_ThermalVias
- SW1, SW2, SW3: footprint Button_Switch_THT:SW_TH_Tactile_Omron_B3F-10xx -> SW_TH_Tactile_Omron_B3F-10xx
- SW_BOOT, SW_RST: footprint Button_Switch_SMD:SW_SPST_B3U-1000P -> SW_SPST_B3U-1000P
- U1: footprint RF_Module:ESP32-S2-MINI-1 -> ESP32-S2-MINI-1
- U_CHG: footprint Package_TO_SOT_SMD:SOT-23-5 -> SOT-23-5
- moved SW_RST 19.5 mm to (185.5, 113.5)
- moved R6 1.00 mm to (173.5, 113.5)
Routing:
- net EN_NET: track 24.4 -> 8.08 mm
- net BOOT_NET: track 26.3 -> 25.3 mm
- net GND: vias 32 -> 29

Commit message: clean gerners now
Parts:
- C1, C3, C7: value C_0603_1608Metric -> 10uF; footprint C_0603_1608Metric -> Capacitor_SMD:C_0603_1608Metric
- C10, C11, C5, C6, C8, C9: value C_0603_1608Metric -> 100nF; footprint C_0603_1608Metric -> Capacitor_SMD:C_0603_1608Metric
- C2: value C_0603_1608Metric -> 22uF; footprint C_0603_1608Metric -> Capacitor_SMD:C_0603_1608Metric
- C4: value C_0603_1608Metric -> 1uF; footprint C_0603_1608Metric -> Capacitor_SMD:C_0603_1608Metric
- D1: value LED_0603_1608Metric -> STAT_LED; footprint LED_0603_1608Metric -> LED_SMD:LED_0603_1608Metric
- J_BAT1: renamed from J_BAT; value JST_PH_S2B-PH-K_1x02_P2.00mm_Horizontal -> BATT_JST-PH-2P; footprint JST_PH_S2B-PH-K_1x02_P2.00mm_Horizontal -> Connector_JST:JST_PH_S2B-PH-K_1x02_P2.00mm_Horizontal
- J_USB1: renamed from J_USB; value USB_C_Receptacle_GCT_USB4105-xx-A_16P_TopMnt_Horizontal -> USB4105-GF-A; footprint USB_C_Receptacle_GCT_USB4105-xx-A_16P_TopMnt_Horizontal -> Connector_USB:USB_C_Receptacle_GCT_USB4105-xx-A_16P_TopMnt_Horizontal
- L1: value L_Bourns-SRN4018 -> 2.2uH; footprint L_Bourns-SRN4018 -> Inductor_SMD:L_Bourns-SRN4018
- MH1, MH2: value MountingHole_4.3mm_M4 -> MountingHole; footprint MountingHole_4.3mm_M4 -> MountingHole:MountingHole_4.3mm_M4
- R1: value R_0603_1608Metric -> 2k; footprint R_0603_1608Metric -> Resistor_SMD:R_0603_1608Metric
- R2: value R_0603_1608Metric -> 1k; footprint R_0603_1608Metric -> Resistor_SMD:R_0603_1608Metric
- R3, R4: value R_0603_1608Metric -> 5.1k; footprint R_0603_1608Metric -> Resistor_SMD:R_0603_1608Metric
- R5, R6: value R_0603_1608Metric -> 10k; footprint R_0603_1608Metric -> Resistor_SMD:R_0603_1608Metric
- R7, R8: value R_0603_1608Metric -> 100k; footprint R_0603_1608Metric -> Resistor_SMD:R_0603_1608Metric
- REG1: value Texas_DRC0010J_ThermalVias -> TPS63001DRCR; footprint Texas_DRC0010J_ThermalVias -> Package_SON:Texas_DRC0010J
- SW1, SW2, SW3: value SW_TH_Tactile_Omron_B3F-10xx -> B3F-100x; footprint SW_TH_Tactile_Omron_B3F-10xx -> Button_Switch_THT:SW_TH_Tactile_Omron_B3F-100x
- SW_BOOT1: renamed from SW_BOOT; value SW_SPST_B3U-1000P -> BOOT; footprint SW_SPST_B3U-1000P -> Button_Switch_SMD:SW_SPST_B3U-1000P
- SW_RST1: renamed from SW_RST; value SW_SPST_B3U-1000P -> RESET; footprint SW_SPST_B3U-1000P -> Button_Switch_SMD:SW_SPST_B3U-1000P
- U1: value ESP32-S2-MINI-1 -> ESP32-S3-MINI-1-N4R2; footprint ESP32-S2-MINI-1 -> RF_Module:ESP32-S2-MINI-1
- U_CHG1: renamed from U_CHG; value SOT-23-5 -> MCP73831T-2ACI/OT; footprint SOT-23-5 -> Package_TO_SOT_SMD:SOT-23-5
- moved SW_RST1 19.5 mm to (166.0, 113.5)
- moved R6 1.00 mm to (172.5, 113.5)
Connections:
- net BOOT_NET renamed /BOOT_NET
- net CHG_PROG renamed /CHG_PROG
- net CHG_STAT renamed /CHG_STAT
- net EN_NET renamed /EN_NET
- net L_A renamed /L_A
- net L_B renamed /L_B
- net STAT_LED_MID renamed /STAT_LED_MID
- net SW1_NET renamed /SW1_NET
- net SW2_NET renamed /SW2_NET
- net SW3_NET renamed /SW3_NET
- net USB_CC1 renamed /USB_CC1
- net USB_CC2 renamed /USB_CC2
- net USB_DM renamed /USB_DM
- net USB_DP renamed /USB_DP
- net VBAT_SENSE renamed /VBAT_SENSE
- J_USB1 pad A8: (no net) -> unconnected-(J_USB1-SBU1-PadA8)
- J_USB1 pad B8: (no net) -> unconnected-(J_USB1-SBU2-PadB8)
- U1 pad 10: (no net) -> unconnected-(U1-IO6-Pad10)
- U1 pad 11: (no net) -> unconnected-(U1-IO7-Pad11)
- U1 pad 12: (no net) -> unconnected-(U1-IO8-Pad12)
- U1 pad 13: (no net) -> unconnected-(U1-IO9-Pad13)
- U1 pad 17: (no net) -> unconnected-(U1-IO13-Pad17)
- U1 pad 18: (no net) -> unconnected-(U1-IO14-Pad18)
- U1 pad 19: (no net) -> unconnected-(U1-IO15-Pad19)
- U1 pad 20: (no net) -> unconnected-(U1-IO16-Pad20)
- U1 pad 21: (no net) -> unconnected-(U1-IO17-Pad21)
- U1 pad 22: (no net) -> unconnected-(U1-IO18-Pad22)
- U1 pad 25: (no net) -> unconnected-(U1-IO21-Pad25)
- U1 pad 26: (no net) -> unconnected-(U1-IO26-Pad26)
- U1 pad 27: (no net) -> unconnected-(U1-IO47-Pad27)
- U1 pad 28: (no net) -> unconnected-(U1-IO33-Pad28)
- U1 pad 29: (no net) -> unconnected-(U1-IO34-Pad29)
- U1 pad 30: (no net) -> unconnected-(U1-IO48-Pad30)
- U1 pad 31: (no net) -> unconnected-(U1-IO35-Pad31)
- U1 pad 32: (no net) -> unconnected-(U1-IO36-Pad32)
- U1 pad 33: (no net) -> unconnected-(U1-IO37-Pad33)
- U1 pad 34: (no net) -> unconnected-(U1-IO38-Pad34)
- U1 pad 35: (no net) -> unconnected-(U1-IO39-Pad35)
- U1 pad 36: (no net) -> unconnected-(U1-IO40-Pad36)
- U1 pad 37: (no net) -> unconnected-(U1-IO41-Pad37)
- U1 pad 38: (no net) -> unconnected-(U1-IO42-Pad38)
- U1 pad 39: (no net) -> unconnected-(U1-TXD0-Pad39)
- U1 pad 40: (no net) -> unconnected-(U1-RXD0-Pad40)
- U1 pad 41: (no net) -> unconnected-(U1-IO45-Pad41)
- U1 pad 44: (no net) -> unconnected-(U1-IO46-Pad44)
- U1 pad 5: (no net) -> unconnected-(U1-IO1-Pad5)
- U1 pad 6: (no net) -> unconnected-(U1-IO2-Pad6)
- U1 pad 7: (no net) -> unconnected-(U1-IO3-Pad7)
- U1 pad 8: (no net) -> unconnected-(U1-IO4-Pad8)
Routing:
- net /EN_NET: track 8.08 -> 24.4 mm
- net /BOOT_NET: track 25.3 -> 26.3 mm
- net GND: vias 29 -> 32
