File: electrical/mechanical_switch/old/RB_Switch.kicad_sch (KiCad schematic)
At the start: 31 parts, among them SW1 B3F-10xx, SW2 B3F-10xx, SW3 B3F-10xx, U1 ESP32-S3-MINI-1-N4R2

Commit message: fixed schematic and pcb errors
Parts:
- REG1: footprint Package_SON:Texas_DRC0010J -> Package_SON:Texas_DRC0010J_ThermalVias
Connections:
- net BOOT_NET: no longer R6.2, SW_BOOT.1, U1.4 (IO0)
- net CHG_PROG: no longer R1.1, U_CHG.5 (PROG)
- net CHG_STAT: no longer D1.1 (K), U_CHG.1 (STAT)
- net EN_NET: no longer R5.2, SW_RST.1, U1.45 (EN)
- net GND: no longer C1.2, C10.2, C11.2, C2.2, C3.2, C4.2, C5.2, C6.2, C7.2, C8.2, C9.2, J_BAT.2 (Pin_2), J_USB.A1 (GND), J_USB.A12 (GND), J_USB.B1 (GND), J_USB.B12 (GND), J_USB.S1 (SHIELD), R1.2, R3.2, R4.2, R8.2, REG1.11 (PGND), REG1.3 (PGND), REG1.7 (PS/SYNC), REG1.9 (GND), SW1.2, SW2.2, SW3.2, SW_BOOT.2, SW_RST.2, U1.1 (GND), U1.2 (GND), U1.42 (GND), U1.43 (GND), U1.46 (GND), U1.47 (GND), U1.48 (GND), U1.49 (GND), U1.50 (GND), U1.51 (GND), U1.52 (GND), U1.53 (GND), U1.54 (GND), U1.55 (GND), U1.56 (GND), U1.57 (GND), U1.58 (GND), U1.59 (GND), U1.60 (GND), U1.61 (GND), U1.62 (GND), U1.63 (GND), U1.64 (GND), U1.65 (GND), U_CHG.2 (V_{SS})
- net L_A: no longer L1.1, REG1.4 (L1)
- net L_B: no longer L1.2, REG1.2 (L2)
- net STAT_LED_MID: no longer D1.2 (A), R2.1
- net SW1_NET: no longer C9.1, SW1.1, U1.14 (IO10)
- net SW2_NET: no longer C10.1, SW2.1, U1.15 (IO11)
- net SW3_NET: no longer C11.1, SW3.1, U1.16 (IO12)
- net USB_CC1: no longer J_USB.A5 (CC1), R3.1
- net USB_CC2: no longer J_USB.B5 (CC2), R4.1
- net USB_DM: no longer J_USB.A7 (D-), J_USB.B7 (D-), U1.23 (IO19)
- net USB_DP: no longer J_USB.A6 (D+), J_USB.B6 (D+), U1.24 (IO20)
- net V3V3: no longer C2.1, C3.1, C5.1, C6.1, C7.1, R2.2, R5.1, R6.1, REG1.1 (VOUT), REG1.10 (FB), U1.3 (3V3)
- net VBAT: no longer C1.1, J_BAT.1 (Pin_1), R7.1, REG1.5 (VIN), REG1.6 (EN), REG1.8 (VINA), U_CHG.3 (V_{BAT})
- net VBAT_SENSE: no longer C8.1, R7.2, R8.1, U1.9 (IO5)
- net VBUS: no longer C4.1, J_USB.A4 (VBUS), J_USB.A9 (VBUS), J_USB.B4 (VBUS), J_USB.B9 (VBUS), U_CHG.4 (V_{DD})

Commit message: clean gerners now
Parts:
- REG1: footprint Package_SON:Texas_DRC0010J_ThermalVias -> Package_SON:Texas_DRC0010J
- SW1, SW2, SW3: value B3F-10xx -> B3F-100x; footprint Button_Switch_THT:SW_TH_Tactile_Omron_B3F-10xx -> Button_Switch_THT:SW_TH_Tactile_Omron_B3F-100x
- renumbered J_BAT to J_BAT1, J_USB to J_USB1, SW_BOOT to SW_BOOT1, SW_RST to SW_RST1, U_CHG to U_CHG1
Connections:
- net BOOT_NET: now also R6.2, SW_BOOT1.1, U1.4 (IO0)
- net CHG_PROG: now also R1.1, U_CHG1.5 (PROG)
- net CHG_STAT: now also D1.1 (K), U_CHG1.1 (STAT)
- net EN_NET: now also R5.2, SW_RST1.1, U1.45 (EN)
- net GND: now also C1.2, C10.2, C11.2, C2.2, C3.2, C4.2, C5.2, C6.2, C7.2, C8.2, C9.2, J_BAT1.2 (Pin_2), J_USB1.A1 (GND), J_USB1.A12 (GND), J_USB1.B1 (GND), J_USB1.B12 (GND), J_USB1.SH (SHIELD), R1.2, R3.2, R4.2, R8.2, REG1.11 (PGND), REG1.3 (PGND), REG1.7 (PS/SYNC), REG1.9 (GND), SW1.2, SW2.2, SW3.2, SW_BOOT1.2, SW_RST1.2, U1.1 (GND), U1.2 (GND), U1.42 (GND), U1.43 (GND), U1.46 (GND), U1.47 (GND), U1.48 (GND), U1.49 (GND), U1.50 (GND), U1.51 (GND), U1.52 (GND), U1.53 (GND), U1.54 (GND), U1.55 (GND), U1.56 (GND), U1.57 (GND), U1.58 (GND), U1.59 (GND), U1.60 (GND), U1.61 (GND), U1.62 (GND), U1.63 (GND), U1.64 (GND), U1.65 (GND), U_CHG1.2 (V_{SS})
- net L_A: now also L1.1, REG1.4 (L1)
- net L_B: now also L1.2, REG1.2 (L2)
- net STAT_LED_MID: now also D1.2 (A), R2.1
- net SW1_NET: now also C9.1, SW1.1, U1.14 (IO10)
- net SW2_NET: now also C10.1, SW2.1, U1.15 (IO11)
- net SW3_NET: now also C11.1, SW3.1, U1.16 (IO12)
- net USB_CC1: now also J_USB1.A5 (CC1), R3.1
- net USB_CC2: now also J_USB1.B5 (CC2), R4.1
- net USB_DM: now also J_USB1.A7 (D-), J_USB1.B7 (D-), U1.23 (IO19)
- net USB_DP: now also J_USB1.A6 (D+), J_USB1.B6 (D+), U1.24 (IO20)
- net V3V3: now also C2.1, C3.1, C5.1, C6.1, C7.1, R2.2, R5.1, R6.1, REG1.1 (VOUT), REG1.10 (FB), U1.3 (3V3)
- net VBAT: now also C1.1, J_BAT1.1 (Pin_1), R7.1, REG1.5 (VIN), REG1.6 (EN), REG1.8 (VINA), U_CHG1.3 (V_{BAT})
- net VBAT_SENSE: now also C8.1, R7.2, R8.1, U1.9 (IO5)
- net VBUS: now also C4.1, J_USB1.A4 (VBUS), J_USB1.A9 (VBUS), J_USB1.B4 (VBUS), J_USB1.B9 (VBUS), U_CHG1.4 (V_{DD})
